File: hw/charger.sch (KiCad schematic (older format))
At the start: 42 parts, among them J2 FC681495, Q1 BSC080N03MS, U3 BQ24192, U4 LTC1871, U5 LTC2941CMS8E

Commit message: updated schematic ERC ok
Parts:
- renumbered C6 to C10, C7 to C11, C8 to C12, C9 to C13, C10 to C14, C11 to C15, C12 to C16, C13 to C17, C14 to C18, C15 to C19, C16 to C20, C17 to C21, C18 to C22, C19 to C23, C20 to C24, C21 to C25, C22 to C26, U3 to U4, U4 to U5, U5 to U6

Commit message: updated schematic
Connections:
- net GND: no longer R18.2, R19.1, U5.3 (FB)
- new net: R18.2, R19.1, U5.3 (FB)
Changed lines of the file:
@@
 	1    0    0    -1
 $EndComp
-Wire Wire Line
-	7100 5650 7100 5700
-Wire Wire Line
-	7100 5600 7100 5650
-Connection ~ 7100 5650
-Wire Wire Line
-	6250 5650 6250 6000
-Wire Wire Line
-	5800 5650 6250 5650
 Text Notes 5750 4800 0    50   ~ 0
 2u2
@@
 Text Notes 600  1300 0    50   ~ 0
 3V9 - 17V
-Connection ~ 6250 5650
-Wire Wire Line
-	6250 5650 7100 5650
 Text HLabel 950  2700 0    50   BiDi ~ 0
 SDA
@@
 Wire Wire Line
 	9200 2550 9200 2600
+Wire Wire Line
+	7100 5600 7100 5650
+Wire Wire Line
+	7100 5650 7100 5700
+Connection ~ 7100 5650
+Wire Wire Line
+	6250 5650 6250 6000
+Wire Wire Line
+	5800 5650 7100 5650
 $EndSCHEMATC

Commit message: updated schematic
Parts:
- J2: footprint (none) -> KLIB_Connector_Power:Cliff_FC681495
Changed lines of the file:
@@
 F 0 "J2" H 1074 1415 50  0000 C CNN
 F 1 "FC681495" H 1074 1324 50  0000 C CNN
-F 2 "" H 1150 1200 50  0001 C CNN
+F 2 "KLIB_Connector_Power:Cliff_FC681495" H 1150 1200 50  0001 C CNN
 F 3 "http://www.cliffuk.co.uk/products/dcconnectors/FC681495.pdf" H 1150 1200 50  0001 C CNN
 	1    1150 1200

Commit message: updated schematic
Parts:
- removed BT1: 2XLP7836140, symbol Device:Battery
- added J3: N42GK-04, KLIB_Connector_Power:N42GK-04, symbol KLIB_Connector_Specialized:N42GK-04
- C10, C11, C22, C24: value 10u/25 -> 10u/25V; footprint (none) -> Capacitor_SMD:C_1210_3225Metric
- C12, C15, C17, C26: footprint (none) -> Capacitor_SMD:C_0805_2012Metric
- C13: footprint (none) -> Capacitor_SMD:C_1206_3216Metric
- C14: value 1u/25V -> 1u/50V; footprint (none) -> Capacitor_SMD:C_0805_2012Metric
- C16, C21, C23: footprint (none) -> Capacitor_SMD:C_1210_3225Metric
- C18: renamed from C19; value 10u -> 10u/25V; footprint (none) -> Capacitor_SMD:C_1210_3225Metric
- C19: renamed from C18; footprint (none) -> Capacitor_SMD:C_1206_3216Metric
- C20: value 10u -> 10u/25V; footprint (none) -> Capacitor_SMD:C_1210_3225Metric
- C25: footprint (none) -> Capacitor_Tantalum_SMD:CP_EIA-7343-31_Kemet-D
- D4, D5: footprint (none) -> LED_SMD:LED_0805_2012Metric
- L1, L2: footprint (none) -> Inductor_SMD:L_12x12mm_H4.5mm
- R10, R11, R12, R13, R14, R15, R16, R17, R18, R19, R8, R9: footprint (none) -> Resistor_SMD:R_0805_2012Metric
- R20: footprint (none) -> Resistor_SMD:R_1206_3216Metric
Connections:
- net GND: now also J3.1, J3.2
- net AKU renamed ACCUPACK+
- net ACCUPACK+: now also J3.3, J3.4
Other:
- note added: "1206"
- note added: "2XLP7836140"
- note removed: "X7R 1211"
- moved on the sheet: C18

Commit message: updated schematic
Parts:
- renumbered D3 to D5, D4 to D6, D5 to D7, D6 to D8, R8 to R14, R9 to R15, R10 to R16, R11 to R17, R12 to R18, R13 to R19, R14 to R20, R15 to R21, R16 to R22, R17 to R23, R18 to R24, R19 to R25, R20 to R26

Commit message: updated schematic
Parts:
- added R27: 10k, Resistor_SMD:R_0805_2012Metric, symbol Device:R
Connections:
- net +3V3: now also R27.1
- net ~AL: now also R27.2
Changed lines of the file:
@@
 Wire Wire Line
 	950  2900 2200 2900
-Text HLabel 10850 2800 2    50   Output ~ 0
+Text HLabel 950  3000 0    50   Output ~ 0
 ~AL
 Wire Wire Line
-	10550 2800 10850 2800
+	10550 2800 10800 2800
 $Comp
 L KLIB_Power:PWR_FLAG #FLG03
@@
 Wire Wire Line
 	9650 4650 9750 4650
+$Comp
+L Device:R R27
+U 1 1 5B030A88
+P 1300 2200
+F 0 "R27" H 1370 2246 50  0000 L CNN
+F 1 "10k" H 1370 2155 50  0000 L CNN
+F 2 "Resistor_SMD:R_0805_2012Metric" V 1230 2200 50  0001 C CNN
+F 3 "~" H 1300 2200 50  0001 C CNN
+	1    1300 2200
+	1    0    0    -1
+$EndComp
+$Comp
+L KLIB_Power:+3V3 #PWR062
+U 1 1 5B03136A
+P 1300 2050
+F 0 "#PWR062" H 1300 1750 50  0001 C CNN
+F 1 "+3V3" H 1305 2223 50  0000 C CNN
+F 2 "" H 1300 2050 50  0001 C CNN
+F 3 "" H 1300 2050 50  0001 C CNN
+	1    1300 2050
+	1    0    0    -1
+$EndComp
+Wire Wire Line
+	950  3000 1300 3000
+Wire Wire Line
+	1300 3000 1300 2350
+Text Label 1050 3000 0    50   ~ 0
+~AL
 $EndSCHEMATC
