File: hw/back.kicad_pcb (KiCad board)
At the start: 2 copper layers, 110 x 55 mm, 77 parts, among them J1 IDC_02X13, J2 FC681495, J3 N42GK-04, Q1 BSC080N03MS, U1 OSRB38C9BA, U2 MCP1826S, U3 MCP1826S, U4 BQ24192, U5 LTC1871, U6 LTC2941CMS8E

Commit message: updated pcb
Parts:
- moved D5 22.1 mm to (175.2, 107.2)
- moved R4 2.02 mm to (123.8, 105.0)
- moved R5 2.02 mm to (123.8, 107.0)
- moved R6 2.02 mm to (123.8, 109.0)
- moved D2 2.00 mm to (130.0, 107.0)
- moved D3 2.00 mm to (160.0, 107.0)
- moved R10 2.00 mm to (166.2, 105.0)
- moved R8 2.00 mm to (166.2, 109.0)
- moved R9 2.00 mm to (166.2, 107.0)
- moved D4 0.20 mm to (190.0, 105.0)
Routing:
- net +5V: track 0.00 -> 34.0 mm
- net Net-(D5-Pad1): track 0.00 -> 25.3 mm
- net +5V5: track 0.00 -> 20.3 mm
- net +3V3: track 0.00 -> 8.25 mm
- net /~AL: track 0.00 -> 5.60 mm
- net /~INT: track 0.00 -> 5.51 mm
- net /SCL: track 0.00 -> 5.43 mm
- net /SDA: track 0.00 -> 5.40 mm
- net Net-(D4-Pad3): track 0.00 -> 3.34 mm
- net Net-(D4-Pad1): track 0.00 -> 3.34 mm
- net Net-(D4-Pad2): track 0.00 -> 3.22 mm
- net Net-(D3-Pad3): track 0.00 -> 3.09 mm
- net Net-(D3-Pad1): track 0.00 -> 3.09 mm
- net Net-(D2-Pad3): track 0.00 -> 3.09 mm
- net Net-(D2-Pad1): track 0.00 -> 3.09 mm
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- added copper zone on B.Cu, net GND
- added copper zone on F.Cu, net GND

Commit message: updated pcb
Routing:
- net +BATT: track 0.00 -> 53.2 mm
- net /charger/ACCUPACK+: track 0.00 -> 20.0 mm
Changed lines of the file:
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@@
     (thickness 1.6)
     (drawings 6)
-    (tracks 78)
+    (tracks 88)
     (zones 0)
     (modules 77)
@@
   )
   (setup
-    (last_trace_width 1)
+    (last_trace_width 0.25)
     (user_trace_width 0.5)
     (user_trace_width 0.8)
@@
     (model ${KISYS3DMOD}/Inductor_SMD.3dshapes/L_12x12mm_H4.5mm.wrl
       (at (xyz 0 0 0))
-      (scale (xyz 1 1 1))
+      (scale (xyz 4 4 4))
       (rotate (xyz 0 0 0))
     )
@@
     (model ${KISYS3DMOD}/Inductor_SMD.3dshapes/L_12x12mm_H4.5mm.wrl
       (at (xyz 0 0 0))
-      (scale (xyz 1 1 1))
+      (scale (xyz 4 4 4))
       (rotate (xyz 0 0 0))
     )
@@
   (gr_line (start 200 85) (end 200 140) (layer Edge.Cuts) (width 0.15))
   (gr_line (start 90 85) (end 200 85) (layer Edge.Cuts) (width 0.15))
+  (segment (start 168.25 127.1) (end 165.15 124) (width 2) (layer F.Cu) (net 1))
+  (segment (start 165.15 124) (end 159.2 124) (width 2) (layer F.Cu) (net 1))
+  (segment (start 159.2 124) (end 157.5 125.7) (width 2) (layer F.Cu) (net 1))
+  (segment (start 157.5 125.7) (end 157.5 127.5) (width 2) (layer F.Cu) (net 1))
+  (segment (start 173.75 127.1) (end 168.25 127.1) (width 2) (layer F.Cu) (net 1))
   (segment (start 111.62 91) (end 111.62 88.46) (width 2) (layer F.Cu) (net 3))
   (segment (start 106.54 91) (end 106.54 88.46) (width 2) (layer F.Cu) (net 3))
@@
   (segment (start 132.5 94.36) (end 131.94 93.8) (width 0.5) (layer F.Cu) (net 29))
   (segment (start 132.5 96.37) (end 132.5 94.36) (width 0.5) (layer F.Cu) (net 29))
+  (segment (start 113.25 111.75) (end 155 111.75) (width 2) (layer F.Cu) (net 31))
+  (segment (start 155 111.75) (end 156.7 113.45) (width 2) (layer F.Cu) (net 31))
+  (segment (start 111.55 113.45) (end 113.25 111.75) (width 2) (layer F.Cu) (net 31))
+  (segment (start 111.55 116.75) (end 111.55 113.45) (width 2) (layer F.Cu) (net 31))
+  (segment (start 156.7 113.45) (end 156.7 116.75) (width 2) (layer F.Cu) (net 31))
   (segment (start 187.6 106.7) (end 184.68 106.7) (width 0.5) (layer F.Cu) (net 45))
   (segment (start 184.68 106.7) (end 184.38 107) (width 0.5) (layer F.Cu) (net 45))

Commit message: updated pcb
Parts:
- moved J3 5.00 mm to (171.0, 120.0)
- moved C26 2.15 mm to (160.2, 134.8)
- moved R26 2.15 mm to (159.2, 130.8)
- moved U6 2.15 mm to (162.5, 130.8)
- moved C18 1.80 mm to (152.5, 126.5)
- moved C20 1.80 mm to (149.2, 126.5)
- moved C21 1.80 mm to (152.5, 133.5)
- moved C23 1.80 mm to (149.2, 133.5)
Routing:
- net /charger/ACCUPACK+: track 20.0 -> 0.00 mm
Changed lines of the file:
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@@
     (thickness 1.6)
     (drawings 6)
-    (tracks 88)
+    (tracks 83)
     (zones 0)
     (modules 77)
@@
   )
   (module Capacitor_SMD:C_0805_2012Metric (layer F.Cu)
-    (at 158.5 133.5 180)
+    (at 160.25 134.75 180)
     (descr "Capacitor SMD 0805 (2012 Metric), square (rectangular) end terminal, IPC_7351 nominal, (Body size source: http://www.tortai-tech.com/upload/download/2011102023233369053.pdf), generated with kicad-footprint-generator")
     (tags capacitor)
@@
   )
   (module Capacitor_SMD:C_1210_3225Metric (layer F.Cu)
-    (at 147.75 127.5 90)
+    (at 149.25 126.5 90)
     (descr "Capacitor SMD 1210 (3225 Metric), square (rectangular) end terminal, IPC_7351 nominal, (Body size source: http://www.tortai-tech.com/upload/download/2011102023233369053.pdf), generated with kicad-footprint-generator")
     (tags capacitor)
@@
   )
   (module Capacitor_SMD:C_1210_3225Metric (layer F.Cu)
-    (at 151 127.5 90)
+    (at 152.5 126.5 90)
     (descr "Capacitor SMD 1210 (3225 Metric), square (rectangular) end terminal, IPC_7351 nominal, (Body size source: http://www.tortai-tech.com/upload/download/2011102023233369053.pdf), generated with kicad-footprint-generator")
     (tags capacitor)
@@
   )
   (module Capacitor_SMD:C_1210_3225Metric (layer F.Cu)
-    (at 151 132.5 270)
+    (at 152.5 133.5 270)
     (descr "Capacitor SMD 1210 (3225 Metric), square (rectangular) end terminal, IPC_7351 nominal, (Body size source: http://www.tortai-tech.com/upload/download/2011102023233369053.pdf), generated with kicad-footprint-generator")
     (tags capacitor)
@@
   )
   (module Capacitor_SMD:C_1210_3225Metric (layer F.Cu)
-    (at 147.75 132.5 270)
+    (at 149.25 133.5 270)
     (descr "Capacitor SMD 1210 (3225 Metric), square (rectangular) end terminal, IPC_7351 nominal, (Body size source: http://www.tortai-tech.com/upload/download/2011102023233369053.pdf), generated with kicad-footprint-generator")
     (tags capacitor)
@@
   )
   (module KLIB_Connector_Power:N42GK-04 (layer F.Cu)
-    (at 171 125 180)
+    (at 171 120 180)
     (descr https://www.tme.eu/cz/details/n42gk-04/signalove-konektory-raster-420mm/ninigi/)
     (tags "N42GK-04 NINIGI MOLEX 2X2")
@@
   )
   (module Package_SO:MSOP-8-1EP_3x3mm_P0.65mm_EP1.68x1.88mm (layer F.Cu)
-    (at 160.75 129.5 90)
+    (at 162.5 130.75 90)
     (descr "MS8E Package; 8-Lead Plastic MSOP, Exposed Die Pad (see Linear Technology 05081662_K_MS8E.pdf)")
     (tags "SSOP 0.65")
@@
   )
   (module Resistor_SMD:R_1206_3216Metric (layer F.Cu)
-    (at 157.5 129.5 270)
+    (at 159.25 130.75 270)
     (descr "Resistor SMD 1206 (3216 Metric), square (rectangular) end terminal, IPC_7351 nominal, (Body size source: http://www.tortai-tech.com/upload/download/2011102023233369053.pdf), generated with kicad-footprint-generator")
     (tags resistor)
@@
   (gr_line (start 200 85) (end 200 140) (layer Edge.Cuts) (width 0.15))
   (gr_line (start 90 85) (end 200 85) (layer Edge.Cuts) (width 0.15))
-  (segment (start 168.25 127.1) (end 165.15 124) (width 2) (layer F.Cu) (net 1))
-  (segment (start 165.15 124) (end 159.2 124) (width 2) (layer F.Cu) (net 1))
-  (segment (start 159.2 124) (end 157.5 125.7) (width 2) (layer F.Cu) (net 1))
-  (segment (start 157.5 125.7) (end 157.5 127.5) (width 2) (layer F.Cu) (net 1))
-  (segment (start 173.75 127.1) (end 168.25 127.1) (width 2) (layer F.Cu) (net 1))
   (segment (start 111.62 91) (end 111.62 88.46) (width 2) (layer F.Cu) (net 3))
   (segment (start 106.54 91) (end 106.54 88.46) (width 2) (layer F.Cu) (net 3))

Commit message: updated pcb
Parts:
- moved C18 1.25 mm to (151.2, 126.5)
- moved C20 1.25 mm to (148.0, 126.5)
- moved C21 1.25 mm to (151.2, 133.5)
- moved C23 1.25 mm to (148.0, 133.5)
Routing:
- net +BATT: track 53.2 -> 79.1 mm
- net /charger/BAT: track 0.00 -> 19.5 mm
- net /charger/ACCUPACK+: track 0.00 -> 18.6 mm
Changed lines of the file:
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@@
     (thickness 1.6)
     (drawings 6)
-    (tracks 83)
+    (tracks 125)
     (zones 0)
     (modules 77)
@@
   )
   (setup
-    (last_trace_width 0.25)
+    (last_trace_width 0.5)
     (user_trace_width 0.5)
     (user_trace_width 0.8)
@@
   )
   (module Capacitor_SMD:C_1210_3225Metric (layer F.Cu)
-    (at 149.25 126.5 90)
+    (at 148 126.5 90)
     (descr "Capacitor SMD 1210 (3225 Metric), square (rectangular) end terminal, IPC_7351 nominal, (Body size source: http://www.tortai-tech.com/upload/download/2011102023233369053.pdf), generated with kicad-footprint-generator")
     (tags capacitor)
@@
   )
   (module Capacitor_SMD:C_1210_3225Metric (layer F.Cu)
-    (at 152.5 126.5 90)
+    (at 151.25 126.5 90)
     (descr "Capacitor SMD 1210 (3225 Metric), square (rectangular) end terminal, IPC_7351 nominal, (Body size source: http://www.tortai-tech.com/upload/download/2011102023233369053.pdf), generated with kicad-footprint-generator")
     (tags capacitor)
@@
   )
   (module Capacitor_SMD:C_1210_3225Metric (layer F.Cu)
-    (at 152.5 133.5 270)
+    (at 151.25 133.5 270)
     (descr "Capacitor SMD 1210 (3225 Metric), square (rectangular) end terminal, IPC_7351 nominal, (Body size source: http://www.tortai-tech.com/upload/download/2011102023233369053.pdf), generated with kicad-footprint-generator")
     (tags capacitor)
@@
   )
   (module Capacitor_SMD:C_1210_3225Metric (layer F.Cu)
-    (at 149.25 133.5 270)
+    (at 148 133.5 270)
     (descr "Capacitor SMD 1210 (3225 Metric), square (rectangular) end terminal, IPC_7351 nominal, (Body size source: http://www.tortai-tech.com/upload/download/2011102023233369053.pdf), generated with kicad-footprint-generator")
     (tags capacitor)
@@
   (gr_line (start 200 85) (end 200 140) (layer Edge.Cuts) (width 0.15))
   (gr_line (start 90 85) (end 200 85) (layer Edge.Cuts) (width 0.15))
+  (segment (start 159.25 129.32) (end 159.25 127.35) (width 2) (layer F.Cu) (net 1))
+  (segment (start 159.25 127.35) (end 164.5 122.1) (width 2) (layer F.Cu) (net 1))
+  (segment (start 164.5 122.1) (end 168.25 122.1) (width 2) (layer F.Cu) (net 1))
+  (segment (start 173.75 122.1) (end 168.25 122.1) (width 2) (layer F.Cu) (net 1))
+  (segment (start 144.299999 130.050001) (end 144.630001 130.380003) (width 0.5) (layer F.Cu) (net 2))
+  (segment (start 144.630001 130.380003) (end 144.630001 130.800001) (width 0.5) (layer F.Cu) (net 2))
+  (segment (start 143.9 130.45) (end 144.299999 130.050001) (width 0.5) (layer F.Cu) (net 2))
+  (segment (start 143.85 130.45) (end 143.9 130.45) (width 0.5) (layer F.Cu) (net 2))
+  (segment (start 144.630001 130.800001) (end 144.300001 130.800001) (width 0.5) (layer F.Cu) (net 2))
+  (segment (start 144.300001 130.800001) (end 143.95 130.45) (width 0.5) (layer F.Cu) (net 2))
+  (segment (start 143.85 130.45) (end 143.95 130.45) (width 0.5) (layer F.Cu) (net 2))
+  (segment (start 143.95 130.45) (end 144.2 130.2) (width 0.5) (layer F.Cu) (net 2))
+  (segment (start 143.650001 130.2) (end 143.650001 130.149999) (width 0.5) (layer F.Cu) (net 2))
+  (segment (start 143.650001 130.149999) (end 143.749993 130.050007) (width 0.5) (layer F.Cu) (net 2))
+  (segment (start 144.2 130.2) (end 143.650001 130.2) (width 0.5) (layer F.Cu) (net 2))
+  (segment (start 144.630001 130.630001) (end 144.2 130.2) (width 0.5) (layer F.Cu) (net 2))
+  (segment (start 144.630001 130.800001) (end 144.630001 130.630001) (width 0.5) (layer F.Cu) (net 2))
+  (segment (start 145.9 132.07) (end 144.630001 130.800001) (width 1.2) (layer F.Cu) (net 2))
+  (segment (start 149.25 132.07) (end 145.9 132.07) (width 2) (layer F.Cu) (net 2))
+  (segment (start 152.5 132.07) (end 159.14 132.07) (width 2) (layer F.Cu) (net 2))
+  (segment (start 159.14 132.07) (end 159.25 132.18) (width 2) (layer F.Cu) (net 2))
+  (segment (start 149.25 132.07) (end 152.5 132.07) (width 2) (layer F.Cu) (net 2))
   (segment (start 111.62 91) (end 111.62 88.46) (width 2) (layer F.Cu) (net 3))
   (segment (start 106.54 91) (end 106.54 88.46) (width 2) (layer F.Cu) (net 3))
@@
   (segment (start 132.5 94.36) (end 131.94 93.8) (width 0.5) (layer F.Cu) (net 29))
   (segment (start 132.5 96.37) (end 132.5 94.36) (width 0.5) (layer F.Cu) (net 29))
+  (segment (start 144.15 129.3) (end 145.2 129.3) (width 0.5) (layer F.Cu) (net 31))
+  (segment (start 145.2 129.3) (end 145.4 129.1) (width 0.5) (layer F.Cu) (net 31))
+  (segment (start 144.6 129.1) (end 144.6 129.15) (width 0.5) (layer F.Cu) (net 31))
+  (segment (start 144.6 129.15) (end 144.75 129.3) (width 0.5) (layer F.Cu) (net 31))
+  (segment (start 144.75 129.3) (end 144.15 129.3) (width 0.5) (layer F.Cu) (net 31))
+  (segment (start 144.6 129.1) (end 145.4 129.1) (width 0.5) (layer F.Cu) (net 31))
+  (segment (start 144.25 129.1) (end 144.6 129.1) (width 0.5) (layer F.Cu) (net 31))
+  (segment (start 144.15 129.2) (end 143.650001 129.2) (width 0.5) (layer F.Cu) (net 31))
+  (segment (start 144.15 129.2) (end 144.15 129.3) (width 0.5) (layer F.Cu) (net 31))
+  (segment (start 144.200001 129.149999) (end 144.25 129.1) (width 0.5) (layer F.Cu) (net 31))
+  (segment (start 143.650001 129.149999) (end 144.200001 129.149999) (width 0.5) (layer F.Cu) (net 31))
+  (segment (start 156.7 116.75) (end 156.7 124.55) (width 2) (layer F.Cu) (net 31))
+  (segment (start 156.7 124.55) (end 153.32 127.93) (width 2) (layer F.Cu) (net 31))
+  (segment (start 153.32 127.93) (end 149.25 127.93) (width 2) (layer F.Cu) (net 31))
+  (segment (start 149.25 127.93) (end 146.57 127.93) (width 2) (layer F.Cu) (net 31))
+  (segment (start 146.57 127.93) (end 145.4 129.1) (width 1.2) (layer F.Cu) (net 31))
+  (segment (start 143.650001 129.2) (end 143.650001 129.250001) (width 0.5) (layer F.Cu) (net 31))
+  (segment (start 143.650001 129.250001) (end 143.749999 129.349999) (width 0.5) (layer F.Cu) (net 31))
+  (segment (start 143.650001 129.2) (end 143.650001 129.149999) (width 0.5) (layer F.Cu) (net 31))
+  (segment (start 143.650001 129.149999) (end 143.749999 129.050001) (width 0.5) (layer F.Cu) (net 31))
   (segment (start 113.25 111.75) (end 155 111.75) (width 2) (layer F.Cu) (net 31))
   (segment (start 155 111.75) (end 156.7 113.45) (width 2) (layer F.Cu) (net 31))

Commit message: updated pcb
Parts:
- moved R26 0.11 mm to (159.2, 130.6)
Routing:
- net +BATT: track 79.1 -> 82.3 mm
- net /charger/BAT: track 19.5 -> 20.7 mm
Changed lines of the file:
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@@
     (thickness 1.6)
     (drawings 6)
-    (tracks 125)
+    (tracks 126)
     (zones 0)
     (modules 77)
@@
   )
   (setup
-    (last_trace_width 0.5)
+    (last_trace_width 2)
     (user_trace_width 0.5)
     (user_trace_width 0.8)
@@
   )
   (module Resistor_SMD:R_1206_3216Metric (layer F.Cu)
-    (at 159.25 130.75 270)
+    (at 159.24 130.64 270)
     (descr "Resistor SMD 1206 (3216 Metric), square (rectangular) end terminal, IPC_7351 nominal, (Body size source: http://www.tortai-tech.com/upload/download/2011102023233369053.pdf), generated with kicad-footprint-generator")
     (tags resistor)
@@
   (gr_line (start 200 85) (end 200 140) (layer Edge.Cuts) (width 0.15))
   (gr_line (start 90 85) (end 200 85) (layer Edge.Cuts) (width 0.15))
-  (segment (start 159.25 129.32) (end 159.25 127.35) (width 2) (layer F.Cu) (net 1))
-  (segment (start 159.25 127.35) (end 164.5 122.1) (width 2) (layer F.Cu) (net 1))
+  (segment (start 159.24 129.21) (end 159.24 127.51) (width 2) (layer F.Cu) (net 1))
+  (segment (start 159.24 127.51) (end 164.5 122.25) (width 2) (layer F.Cu) (net 1))
+  (segment (start 164.5 122.25) (end 164.5 122.1) (width 2) (layer F.Cu) (net 1))
   (segment (start 164.5 122.1) (end 168.25 122.1) (width 2) (layer F.Cu) (net 1))
   (segment (start 173.75 122.1) (end 168.25 122.1) (width 2) (layer F.Cu) (net 1))
+  (segment (start 151.25 132.07) (end 159.24 132.07) (width 2) (layer F.Cu) (net 2))
   (segment (start 144.299999 130.050001) (end 144.630001 130.380003) (width 0.5) (layer F.Cu) (net 2))
   (segment (start 144.630001 130.380003) (end 144.630001 130.800001) (width 0.5) (layer F.Cu) (net 2))
@@
   (segment (start 145.9 132.07) (end 144.630001 130.800001) (width 1.2) (layer F.Cu) (net 2))
   (segment (start 149.25 132.07) (end 145.9 132.07) (width 2) (layer F.Cu) (net 2))
-  (segment (start 152.5 132.07) (end 159.14 132.07) (width 2) (layer F.Cu) (net 2))
-  (segment (start 159.14 132.07) (end 159.25 132.18) (width 2) (layer F.Cu) (net 2))
   (segment (start 149.25 132.07) (end 152.5 132.07) (width 2) (layer F.Cu) (net 2))
   (segment (start 111.62 91) (end 111.62 88.46) (width 2) (layer F.Cu) (net 3))
@@
   (segment (start 132.5 94.36) (end 131.94 93.8) (width 0.5) (layer F.Cu) (net 29))
   (segment (start 132.5 96.37) (end 132.5 94.36) (width 0.5) (layer F.Cu) (net 29))
+  (segment (start 148 127.93) (end 151.25 127.93) (width 0.5) (layer F.Cu) (net 31))
   (segment (start 144.15 129.3) (end 145.2 129.3) (width 0.5) (layer F.Cu) (net 31))
   (segment (start 145.2 129.3) (end 145.4 129.1) (width 0.5) (layer F.Cu) (net 31))
