File: hw/back.kicad_pcb (KiCad board)
At the start: 2 copper layers, 110 x 55 mm, 77 parts, among them J1 IDC_02X13, J2 FC681495, J3 N42GK-04, Q1 BSC080N03MS, U1 OSRB38C9BA, U2 MCP1826S, U3 MCP1826S, U4 BQ24192, U5 LTC1871, U6 LTC2941CMS8E

Commit message: updated pcb
Parts:
- moved C16 1.58 mm to (136.0, 122.5)
- moved C14 1.52 mm to (135.5, 126.0)
- moved C18 1.50 mm to (152.8, 126.5)
- moved C20 1.50 mm to (149.5, 126.5)
- moved C21 1.50 mm to (152.8, 133.5)
- moved C23 1.50 mm to (149.5, 133.5)
- moved C17 0.50 mm to (143.0, 123.0)
- moved C19 0.50 mm to (140.8, 123.0)
Routing:
- net Net-(C17-Pad1): track 0.00 -> 16.8 mm
- net /charger/BAT: track 20.7 -> 25.4 mm
- net +BATT: track 82.3 -> 83.8 mm
Changed lines of the file:
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@@
     (thickness 1.6)
     (drawings 6)
-    (tracks 126)
+    (tracks 146)
     (zones 0)
     (modules 77)
@@
   )
   (setup
-    (last_trace_width 2)
+    (last_trace_width 0.5)
     (user_trace_width 0.5)
     (user_trace_width 0.8)
@@
   )
   (module Capacitor_SMD:C_0805_2012Metric (layer F.Cu)
-    (at 137 125.75 180)
+    (at 135.5 126 180)
     (descr "Capacitor SMD 0805 (2012 Metric), square (rectangular) end terminal, IPC_7351 nominal, (Body size source: http://www.tortai-tech.com/upload/download/2011102023233369053.pdf), generated with kicad-footprint-generator")
     (tags capacitor)
@@
   )
   (module Capacitor_SMD:C_0805_2012Metric (layer F.Cu)
-    (at 143.5 123 270)
+    (at 143 123 270)
     (descr "Capacitor SMD 0805 (2012 Metric), square (rectangular) end terminal, IPC_7351 nominal, (Body size source: http://www.tortai-tech.com/upload/download/2011102023233369053.pdf), generated with kicad-footprint-generator")
     (tags capacitor)
@@
   )
   (module Capacitor_SMD:C_1206_3216Metric (layer F.Cu)
-    (at 141.25 123 90)
+    (at 140.75 123 90)
     (descr "Capacitor SMD 1206 (3216 Metric), square (rectangular) end terminal, IPC_7351 nominal, (Body size source: http://www.tortai-tech.com/upload/download/2011102023233369053.pdf), generated with kicad-footprint-generator")
     (tags capacitor)
@@
   )
   (module Capacitor_SMD:C_1210_3225Metric (layer F.Cu)
-    (at 148 126.5 90)
+    (at 149.5 126.5 90)
     (descr "Capacitor SMD 1210 (3225 Metric), square (rectangular) end terminal, IPC_7351 nominal, (Body size source: http://www.tortai-tech.com/upload/download/2011102023233369053.pdf), generated with kicad-footprint-generator")
     (tags capacitor)
@@
   )
   (module Capacitor_SMD:C_1210_3225Metric (layer F.Cu)
-    (at 151.25 126.5 90)
+    (at 152.75 126.5 90)
     (descr "Capacitor SMD 1210 (3225 Metric), square (rectangular) end terminal, IPC_7351 nominal, (Body size source: http://www.tortai-tech.com/upload/download/2011102023233369053.pdf), generated with kicad-footprint-generator")
     (tags capacitor)
@@
   )
   (module Capacitor_SMD:C_1210_3225Metric (layer F.Cu)
-    (at 137.5 123 180)
+    (at 136 122.5 180)
     (descr "Capacitor SMD 1210 (3225 Metric), square (rectangular) end terminal, IPC_7351 nominal, (Body size source: http://www.tortai-tech.com/upload/download/2011102023233369053.pdf), generated with kicad-footprint-generator")
     (tags capacitor)
@@
   )
   (module Capacitor_SMD:C_1210_3225Metric (layer F.Cu)
-    (at 151.25 133.5 270)
+    (at 152.75 133.5 270)
     (descr "Capacitor SMD 1210 (3225 Metric), square (rectangular) end terminal, IPC_7351 nominal, (Body size source: http://www.tortai-tech.com/upload/download/2011102023233369053.pdf), generated with kicad-footprint-generator")
     (tags capacitor)
@@
   )
   (module Capacitor_SMD:C_1210_3225Metric (layer F.Cu)
-    (at 148 133.5 270)
+    (at 149.5 133.5 270)
     (descr "Capacitor SMD 1210 (3225 Metric), square (rectangular) end terminal, IPC_7351 nominal, (Body size source: http://www.tortai-tech.com/upload/download/2011102023233369053.pdf), generated with kicad-footprint-generator")
     (tags capacitor)
@@
   (segment (start 164.5 122.1) (end 168.25 122.1) (width 2) (layer F.Cu) (net 1))
   (segment (start 173.75 122.1) (end 168.25 122.1) (width 2) (layer F.Cu) (net 1))
+  (segment (start 152.75 132.07) (end 151.25 132.07) (width 0.5) (layer F.Cu) (net 2))
+  (segment (start 149.5 132.07) (end 152.75 132.07) (width 0.5) (layer F.Cu) (net 2))
   (segment (start 151.25 132.07) (end 159.24 132.07) (width 2) (layer F.Cu) (net 2))
   (segment (start 144.299999 130.050001) (end 144.630001 130.380003) (width 0.5) (layer F.Cu) (net 2))
@@
   (segment (start 132.5 94.36) (end 131.94 93.8) (width 0.5) (layer F.Cu) (net 29))
   (segment (start 132.5 96.37) (end 132.5 94.36) (width 0.5) (layer F.Cu) (net 29))
+  (segment (start 149.5 127.93) (end 148 127.93) (width 0.5) (layer F.Cu) (net 31))
   (segment (start 148 127.93) (end 151.25 127.93) (width 0.5) (layer F.Cu) (net 31))
   (segment (start 144.15 129.3) (end 145.2 129.3) (width 0.5) (layer F.Cu) (net 31))
@@
   (segment (start 111.55 116.75) (end 111.55 113.45) (width 2) (layer F.Cu) (net 31))
   (segment (start 156.7 113.45) (end 156.7 116.75) (width 2) (layer F.Cu) (net 31))
+  (segment (start 143.249999 127.349999) (end 143.500001 127.099997) (width 0.5) (layer F.Cu) (net 32))
+  (segment (start 143.500001 127.099997) (end 143.500001 126.499999) (width 0.5) (layer F.Cu) (net 32))
+  (segment (start 143.15 127.25) (end 143.249999 127.349999) (width 0.5) (layer F.Cu) (net 32))
+  (segment (start 142.750001 126.66) (end 142.750001 127.25) (width 0.5) (layer F.Cu) (net 32))
+  (segment (start 142.84 126.66) (end 142.750001 126.66) (width 0.5) (layer F.Cu) (net 32))
+  (segment (start 143.000001 126.499999) (end 142.84 126.66) (width 0.5) (layer F.Cu) (net 32))
+  (segment (start 143.500001 126.499999) (end 143.000001 126.499999) (width 0.5) (layer F.Cu) (net 32))
+  (segment (start 142.980001 126.499999) (end 142.750001 126.729999) (width 0.5) (layer F.Cu) (net 32))
+  (segment (start 143.500001 126.499999) (end 142.980001 126.499999) (width 0.5) (layer F.Cu) (net 32))
+  (segment (start 142.92 127.42) (end 142.82 127.42) (width 0.5) (layer F.Cu) (net 32))
+  (segment (start 142.82 127.42) (end 142.750001 127.350001) (width 0.5) (layer F.Cu) (net 32))
+  (segment (start 143.500001 126.839999) (end 142.92 127.42) (width 0.5) (layer F.Cu) (net 32))
+  (segment (start 143.500001 126.499999) (end 143.500001 126.839999) (width 0.5) (layer F.Cu) (net 32))
+  (segment (start 143.500001 126.499999) (end 143.400001 126.499999) (width 0.5) (layer F.Cu) (net 32))
+  (segment (start 143.400001 126.499999) (end 142.750001 127.149999) (width 0.5) (layer F.Cu) (net 32))
+  (segment (start 146.8 123.2) (end 143.500001 126.499999) (width 2) (layer F.Cu) (net 32))
+  (segment (start 146.8 116.75) (end 146.8 123.2) (width 2) (layer F.Cu) (net 32))
   (segment (start 187.6 106.7) (end 184.68 106.7) (width 0.5) (layer F.Cu) (net 45))
   (segment (start 184.68 106.7) (end 184.38 107) (width 0.5) (layer F.Cu) (net 45))

Commit message: updated pcb
Routing:
- net /charger/ADAPTER: track 0.00 -> 190.8 mm, vias 0 -> 14
- net +BATT: track 83.8 -> 86.1 mm

Commit message: updated pcb
Parts:
- moved C26 1.27 mm to (159.0, 135.0)
Routing:
- net GND: track 0.00 -> 11.1 mm
- net Net-(R22-Pad2): track 0.00 -> 7.63 mm
- net /charger/BAT: track 25.4 -> 31.8 mm
- net /charger/ACCUPACK+: track 18.5 -> 21.7 mm
Changed lines of the file:
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@@
     (thickness 1.6)
     (drawings 6)
-    (tracks 232)
+    (tracks 264)
     (zones 0)
     (modules 77)
@@
   )
   (setup
-    (last_trace_width 2)
+    (last_trace_width 0.25)
     (user_trace_width 0.5)
     (user_trace_width 0.8)
@@
   )
   (module Capacitor_SMD:C_0805_2012Metric (layer F.Cu)
-    (at 160.25 134.75 180)
+    (at 159 135 180)
     (descr "Capacitor SMD 0805 (2012 Metric), square (rectangular) end terminal, IPC_7351 nominal, (Body size source: http://www.tortai-tech.com/upload/download/2011102023233369053.pdf), generated with kicad-footprint-generator")
     (tags capacitor)
@@
   (gr_line (start 200 85) (end 200 140) (layer Edge.Cuts) (width 0.15))
   (gr_line (start 90 85) (end 200 85) (layer Edge.Cuts) (width 0.15))
+  (segment (start 161.525 128.645) (end 161.525 129.35) (width 0.25) (layer F.Cu) (net 1))
+  (segment (start 161.325 129.55) (end 159.58 129.55) (width 0.25) (layer F.Cu) (net 1))
+  (segment (start 159.58 129.55) (end 159.24 129.21) (width 0.25) (layer F.Cu) (net 1))
+  (segment (start 161.525 129.35) (end 161.325 129.55) (width 0.25) (layer F.Cu) (net 1))
+  (segment (start 164.65 122.1) (end 159.24 127.51) (width 2) (layer F.Cu) (net 1))
+  (segment (start 159.88 135) (end 160.69 135) (width 0.25) (layer F.Cu) (net 2))
+  (segment (start 160.69 135) (end 161.525 134.165) (width 0.25) (layer F.Cu) (net 2))
+  (segment (start 161.525 134.165) (end 161.525 133.55) (width 0.25) (layer F.Cu) (net 2))
+  (segment (start 161.525 133.55) (end 161.525 132.855) (width 0.25) (layer F.Cu) (net 2))
+  (segment (start 161.525 132.855) (end 161.525 132.16) (width 0.25) (layer F.Cu) (net 2))
+  (segment (start 159.335 131.975) (end 159.24 132.07) (width 0.25) (layer F.Cu) (net 2))
+  (segment (start 161.525 132.16) (end 161.34 131.975) (width 0.25) (layer F.Cu) (net 2))
+  (segment (start 161.34 131.975) (end 159.335 131.975) (width 0.25) (layer F.Cu) (net 2))
+  (segment (start 141.15 131.15) (end 141.15 129.95) (width 0.25) (layer F.Cu) (net 5))
+  (segment (start 141.15 129.95) (end 141.9 129.2) (width 0.25) (layer F.Cu) (net 5))
+  (segment (start 141.65 131.15) (end 141.65 129.45) (width 0.25) (layer F.Cu) (net 5))
+  (segment (start 141.65 129.45) (end 141.9 129.2) (width 0.25) (layer F.Cu) (net 5))
+  (segment (start 143.610002 127.95) (end 143.560001 128.000001) (width 0.25) (layer F.Cu) (net 5))
+  (segment (start 143.560001 128.000001) (end 142.999999 128.000001) (width 0.25) (layer F.Cu) (net 5))
+  (segment (start 142.999999 128.000001) (end 141.9 129.1) (width 0.25) (layer F.Cu) (net 5))
+  (segment (start 141.9 129.1) (end 141.9 129.2) (width 0.25) (layer F.Cu) (net 5))
+  (segment (start 139.95 128.45) (end 141.15 128.45) (width 0.25) (layer F.Cu) (net 5))
+  (segment (start 141.15 128.45) (end 141.9 129.2) (width 0.25) (layer F.Cu) (net 5))
+  (segment (start 143.85 128.45) (end 142.65 128.45) (width 0.25) (layer F.Cu) (net 5))
+  (segment (start 142.65 128.45) (end 141.9 129.2) (width 0.25) (layer F.Cu) (net 5))
   (segment (start 170 110) (end 153 110) (width 2) (layer B.Cu) (net 24))
   (segment (start 153 110) (end 137.5 125.5) (width 2) (layer B.Cu) (net 24))
@@
   (via (at 137.5 125.5) (size 0.8) (drill 0.4) (layers F.Cu B.Cu) (net 24))
   (segment (start 168.25 122.1) (end 164.65 122.1) (width 2) (layer F.Cu) (net 1))
-  (segment (start 164.65 122.1) (end 159.24 127.51) (width 2) (layer F.Cu) (net 1))
   (segment (start 159.24 127.51) (end 159.24 129.21) (width 2) (layer F.Cu) (net 1))
   (segment (start 173.75 122.1) (end 168.25 122.1) (width 2) (layer F.Cu) (net 1))
@@
   (segment (start 146.8 123.2) (end 143.500001 126.499999) (width 2) (layer F.Cu) (net 32))
   (segment (start 146.8 116.75) (end 146.8 123.2) (width 2) (layer F.Cu) (net 32))
+  (segment (start 143.15 131.15) (end 142.65 131.15) (width 0.25) (layer F.Cu) (net 39))
+  (segment (start 142.65 131.15) (end 142.65 132.6) (width 0.25) (layer F.Cu) (net 39))
+  (segment (start 142.65 132.6) (end 142.25 133) (width 0.25) (layer F.Cu) (net 39))
+  (segment (start 142.25 133) (end 142.25 134.12) (width 0.25) (layer F.Cu) (net 39))
+  (segment (start 143.15 131.15) (end 143.15 131.9) (width 0.25) (layer F.Cu) (net 39))
+  (segment (start 143.15 131.9) (end 144.25 133) (width 0.25) (layer F.Cu) (net 39))
+  (segment (start 144.25 133) (end 144.25 134.12) (width 0.25) (layer F.Cu) (net 39))
+  (segment (start 142.65 133.72) (end 142.25 134.12) (width 0.25) (layer F.Cu) (net 39))
   (segment (start 187.6 106.7) (end 184.68 106.7) (width 0.5) (layer F.Cu) (net 45))
   (segment (start 184.68 106.7) (end 184.38 107) (width 0.5) (layer F.Cu) (net 45))
