File: hw/back.kicad_pcb (KiCad board)
At the start: 2 copper layers, 110 x 55 mm, 77 parts, among them J1 IDC_02X13, J2 FC681495, J3 N42GK-04, Q1 BSC080N03MS, U1 OSRB38C9BA, U2 MCP1826S, U3 MCP1826S, U4 BQ24192, U5 LTC1871, U6 LTC2941CMS8E

Commit message: updated pcb
Parts:
- moved D6 6.52 mm to (129.0, 122.0)
- moved D7 6.52 mm to (131.5, 122.0)
- moved C10 5.40 mm to (101.5, 113.5), turned to 180 degrees
- moved C11 5.06 mm to (101.5, 117.0), turned to 180 degrees
- moved C12 3.04 mm to (103.2, 121.8), turned to 180 degrees
- moved C16 2.06 mm to (138.0, 122.0), turned to 90 degrees
- moved C17 1.03 mm to (143.2, 122.0)
- moved C19 1.03 mm to (141.0, 122.0)
- moved C15 0.25 mm to (99.5, 121.8)
- moved R19 0.25 mm to (99.5, 123.8)
- moved R20 0.25 mm to (99.5, 125.8)
Routing:
- net +BATT: track 86.1 -> 118.2 mm
- net Net-(C19-Pad1): track 0.00 -> 17.8 mm, vias 0 -> 2
- net Net-(D6-Pad1): track 0.00 -> 10.9 mm
- net Net-(D7-Pad1): track 0.00 -> 8.39 mm
- net Net-(C16-Pad1): track 0.00 -> 5.52 mm
- net Net-(R17-Pad1): track 0.00 -> 4.84 mm
- net Net-(C17-Pad2): track 0.00 -> 4.83 mm
- net Net-(R21-Pad1): track 0.00 -> 4.20 mm
- net Net-(R19-Pad1): track 0.00 -> 4.08 mm
- net Net-(R18-Pad1): track 0.00 -> 3.80 mm
- net Net-(C17-Pad1): track 16.8 -> 20.4 mm
- net Net-(R20-Pad1): track 0.00 -> 3.42 mm
- net Net-(C15-Pad1): track 0.00 -> 2.00 mm
- added copper zone on F.Cu, net +BATT

Commit message: updated pcb
Routing:
- net Net-(D8-Pad1): track 0.00 -> 11.2 mm
- net +5V5: track 20.3 -> 23.7 mm
- added copper zone on F.Cu, net +5V5
- added copper zone on F.Cu, net Net-(D8-Pad1)
Changed lines of the file:
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@@
     (thickness 1.6)
     (drawings 6)
-    (tracks 323)
+    (tracks 339)
     (zones 0)
     (modules 77)
@@
   )
   (setup
-    (last_trace_width 1)
+    (last_trace_width 0.25)
     (user_trace_width 0.5)
     (user_trace_width 0.8)
@@
   (segment (start 161.525 132.16) (end 161.34 131.975) (width 0.25) (layer F.Cu) (net 2))
   (segment (start 161.34 131.975) (end 159.335 131.975) (width 0.25) (layer F.Cu) (net 2))
+  (segment (start 104.05 126.25) (end 104.6 126.25) (width 0.25) (layer F.Cu) (net 3))
+  (segment (start 104.6 126.25) (end 104.82 126.47) (width 0.25) (layer F.Cu) (net 3))
+  (segment (start 104.82 126.47) (end 104.82 127.85) (width 0.25) (layer F.Cu) (net 3))
+  (segment (start 104.82 127.85) (end 104.82 129) (width 0.25) (layer F.Cu) (net 3))
   (segment (start 141.15 131.15) (end 141.15 129.95) (width 0.25) (layer F.Cu) (net 5))
   (segment (start 141.15 129.95) (end 141.9 129.2) (width 0.25) (layer F.Cu) (net 5))
@@
   (segment (start 165.07 105.3) (end 165.37 105) (width 0.5) (layer F.Cu) (net 47))
   (segment (start 162.4 107) (end 165.37 107) (width 0.5) (layer F.Cu) (net 48))
+  (segment (start 119.25 127.39) (end 120.15 127.39) (width 0.5) (layer F.Cu) (net 49))
+  (segment (start 120.15 127.39) (end 120.29 127.25) (width 0.5) (layer F.Cu) (net 49))
+  (segment (start 120.31 128.5) (end 120.75 128.5) (width 0.5) (layer F.Cu) (net 49))
+  (segment (start 119.25 128.66) (end 120.15 128.66) (width 0.5) (layer F.Cu) (net 49))
+  (segment (start 120.15 128.66) (end 120.31 128.5) (width 0.5) (layer F.Cu) (net 49))
+  (segment (start 119.25 128.66) (end 118.91 128.66) (width 0.5) (layer F.Cu) (net 49))
+  (segment (start 118.91 128.66) (end 117 126.75) (width 0.5) (layer F.Cu) (net 49))
+  (segment (start 119.25 127.39) (end 117.64 127.39) (width 0.5) (layer F.Cu) (net 49))
+  (segment (start 117.64 127.39) (end 117 126.75) (width 0.5) (layer F.Cu) (net 49))
+  (segment (start 119.25 126.11) (end 120.15 126.11) (width 0.5) (layer F.Cu) (net 49))
+  (segment (start 120.15 126.11) (end 120.26 126) (width 0.5) (layer F.Cu) (net 49))
+  (segment (start 119.25 124.84) (end 121.16 124.84) (width 0.5) (layer F.Cu) (net 49))
   (zone (net 5) (net_name GND) (layer F.Cu) (hatch edge 0.508)
     (connect_pads (clearance 0.508))
@@
       )
     )
+  )
+  (zone (net 49) (net_name "Net-(D8-Pad1)") (layer F.Cu) (hatch edge 0.508)
+    (priority 2)
+    (connect_pads (clearance 0.508))
+    (min_thickness 0.254)
+    (fill yes (arc_segments 16) (thermal_gap 0.508) (thermal_bridge_width 0.508))
+    (polygon
+      (pts
+        (xy 114.75 113.25) (xy 125.25 113.25) (xy 125.25 129.5) (xy 114.75 129.5)
+      )
+    )
+  )
+  (zone (net 3) (net_name +5V5) (layer F.Cu) (hatch edge 0.508)
+    (priority 3)
+    (connect_pads (clearance 0.508))
+    (min_thickness 0.254)
+    (fill yes (arc_segments 16) (thermal_gap 0.508) (thermal_bridge_width 0.508))
+    (polygon
+      (pts
+        (xy 120.75 133.25) (xy 120.75 129.75) (xy 125.25 129.75) (xy 125.25 136.25) (xy 105 136.25)
+        (xy 105 131.75) (xy 101.25 131.75) (xy 101.25 129.5) (xy 103.75 129.5) (xy 103.75 127.5)
+        (xy 106.25 127.5) (xy 106.25 131.25) (xy 108.75 131.25) (xy 108.75 133.25)
+      )
+    )

Commit message: updated pcb
Routing:
- net Net-(D8-Pad1): track 11.2 -> 27.3 mm
- net Net-(R24-Pad2): track 0.00 -> 7.88 mm, vias 0 -> 2
- net Net-(Q1-Pad4): track 0.00 -> 7.68 mm
- net +5V5: track 23.7 -> 27.7 mm, vias 0 -> 15
- net GND: track 11.1 -> 11.8 mm, vias 0 -> 20
- added copper zone on B.Cu, net +5V5

Commit message: updated pcb
Routing:
- net +BATT: track 118.2 -> 20.3 mm
Changed lines of the file:
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@@
     (thickness 1.6)
     (drawings 6)
-    (tracks 406)
+    (tracks 381)
     (zones 0)
     (modules 77)
@@
     (mod_text_size 1 1)
     (mod_text_width 0.15)
-    (pad_size 1.22 2.7)
+    (pad_size 0.85 0.3)
     (pad_drill 0)
     (pad_to_mask_clearance 0.2)
@@
       (net 2 /charger/BAT))
     (pad 15 smd rect (at 1.95 0.25) (size 0.85 0.3) (layers F.Cu F.Paste F.Mask)
-      (net 31 +BATT))
+      (net 31 +BATT) (zone_connect 2))
     (pad 16 smd rect (at 1.95 -0.25) (size 0.85 0.3) (layers F.Cu F.Paste F.Mask)
-      (net 31 +BATT))
+      (net 31 +BATT) (zone_connect 2))
     (pad 17 smd rect (at 1.95 -0.75) (size 0.85 0.3) (layers F.Cu F.Paste F.Mask)
       (net 5 GND))
@@
   (segment (start 132.5 94.36) (end 131.94 93.8) (width 0.5) (layer F.Cu) (net 29))
   (segment (start 132.5 96.37) (end 132.5 94.36) (width 0.5) (layer F.Cu) (net 29))
-  (segment (start 102.93 117) (end 111.3 117) (width 1) (layer F.Cu) (net 31))
+  (segment (start 143.85 129.45) (end 143.85 128.95) (width 0.25) (layer F.Cu) (net 31))
+  (segment (start 144.4 129) (end 144.1 129) (width 0.25) (layer F.Cu) (net 31))
+  (segment (start 144.1 129) (end 143.85 129.25) (width 0.25) (layer F.Cu) (net 31))
+  (segment (start 144.45 128.95) (end 144.4 129) (width 0.25) (layer F.Cu) (net 31))
+  (segment (start 143.85 128.95) (end 144.45 128.95) (width 0.25) (layer F.Cu) (net 31))
+  (segment (start 143.85 129.25) (end 144.75 129.25) (width 0.25) (layer F.Cu) (net 31))
+  (segment (start 143.85 129.45) (end 143.85 129.25) (width 0.25) (layer F.Cu) (net 31))
+  (segment (start 143.85 129.45) (end 144.8 129.45) (width 0.25) (layer F.Cu) (net 31))
+  (segment (start 143.85 128.95) (end 144.525 128.95) (width 0.25) (layer F.Cu) (net 31))
+  (segment (start 144.525 128.95) (end 145.225 128.25) (width 0.25) (layer F.Cu) (net 31))
   (segment (start 111.3 117) (end 111.55 116.75) (width 1) (layer F.Cu) (net 31))
-  (segment (start 102.93 113.5) (end 102.93 117) (width 1) (layer F.Cu) (net 31))
-  (segment (start 103.5 119.42) (end 103 119.42) (width 1) (layer F.Cu) (net 31))
-  (segment (start 103 119.42) (end 102.93 119.35) (width 1) (layer F.Cu) (net 31))
-  (segment (start 102.93 119.35) (end 102.93 117) (width 1) (layer F.Cu) (net 31))
-  (segment (start 104.13 121.75) (end 104.13 120.05) (width 1) (layer F.Cu) (net 31))
-  (segment (start 104.13 120.05) (end 103.5 119.42) (width 1) (layer F.Cu) (net 31))
   (segment (start 104.05 124.25) (end 104.05 121.83) (width 0.25) (layer F.Cu) (net 31))
   (segment (start 104.05 121.83) (end 104.13 121.75) (width 0.25) (layer F.Cu) (net 31))
   (segment (start 129 121.12) (end 129.95 121.12) (width 0.25) (layer F.Cu) (net 31))
   (segment (start 129.95 121.12) (end 131.5 121.12) (width 0.25) (layer F.Cu) (net 31))
-  (segment (start 113.25 111.75) (end 131.5 111.75) (width 2) (layer F.Cu) (net 31))
-  (segment (start 131.5 111.75) (end 155 111.75) (width 2) (layer F.Cu) (net 31))
   (segment (start 131.5 121.12) (end 131.5 111.75) (width 0.25) (layer F.Cu) (net 31))
-  (segment (start 152.75 127.93) (end 148 127.93) (width 0.5) (layer F.Cu) (net 31))
-  (segment (start 148 127.93) (end 149.5 127.93) (width 0.5) (layer F.Cu) (net 31))
-  (segment (start 156.7 116.75) (end 156.7 125.8) (width 2) (layer F.Cu) (net 31))
-  (segment (start 156.7 125.8) (end 154.57 127.93) (width 2) (layer F.Cu) (net 31))
-  (segment (start 154.57 127.93) (end 149.25 127.93) (width 2) (layer F.Cu) (net 31))
-  (segment (start 149.25 127.93) (end 146.57 127.93) (width 2) (layer F.Cu) (net 31))
-  (segment (start 144.15 129.3) (end 145.2 129.3) (width 0.5) (layer F.Cu) (net 31))
-  (segment (start 145.2 129.3) (end 145.4 129.1) (width 0.5) (layer F.Cu) (net 31))
-  (segment (start 144.6 129.1) (end 144.6 129.15) (width 0.5) (layer F.Cu) (net 31))
-  (segment (start 144.6 129.15) (end 144.75 129.3) (width 0.5) (layer F.Cu) (net 31))
-  (segment (start 144.75 129.3) (end 144.15 129.3) (width 0.5) (layer F.Cu) (net 31))
-  (segment (start 144.6 129.1) (end 145.4 129.1) (width 0.5) (layer F.Cu) (net 31))
-  (segment (start 144.25 129.1) (end 144.6 129.1) (width 0.5) (layer F.Cu) (net 31))
-  (segment (start 144.15 129.2) (end 143.650001 129.2) (width 0.5) (layer F.Cu) (net 31))
-  (segment (start 144.15 129.2) (end 144.15 129.3) (width 0.5) (layer F.Cu) (net 31))
-  (segment (start 144.200001 129.149999) (end 144.25 129.1) (width 0.5) (layer F.Cu) (net 31))
-  (segment (start 143.650001 129.149999) (end 144.200001 129.149999) (width 0.5) (layer F.Cu) (net 31))
-  (segment (start 146.57 127.93) (end 145.4 129.1) (width 1.2) (layer F.Cu) (net 31))
-  (segment (start 143.650001 129.2) (end 143.650001 129.250001) (width 0.5) (layer F.Cu) (net 31))
-  (segment (start 143.650001 129.250001) (end 143.749999 129.349999) (width 0.5) (layer F.Cu) (net 31))
-  (segment (start 143.650001 129.2) (end 143.650001 129.149999) (width 0.5) (layer F.Cu) (net 31))
-  (segment (start 143.650001 129.149999) (end 143.749999 129.050001) (width 0.5) (layer F.Cu) (net 31))
-  (segment (start 155 111.75) (end 156.7 113.45) (width 2) (layer F.Cu) (net 31))
-  (segment (start 111.55 113.45) (end 113.25 111.75) (width 2) (layer F.Cu) (net 31))
-  (segment (start 111.55 116.75) (end 111.55 113.45) (width 2) (layer F.Cu) (net 31))
-  (segment (start 156.7 113.45) (end 156.7 116.75) (width 2) (layer F.Cu) (net 31))
   (segment (start 146.8 121.25) (end 146.8 123.2) (width 2) (layer F.Cu) (net 32))
   (segment (start 146.8 116.75) (end 146.8 121.25) (width 2) (layer F.Cu) (net 32))
@@
     (polygon
       (pts
-        (xy 102.25 111.75) (xy 103.25 110.75) (xy 116.5 110.75) (xy 114.25 113) (xy 114.25 119.5)
-        (xy 113.5 120.25) (xy 109 120.25) (xy 109 123.25) (xy 103.5 123.25) (xy 103.5 120.25)
-        (xy 102.25 120.25)
+        (xy 102.25 111.75) (xy 103.25 110.75) (xy 156.75 110.75) (xy 159.75 113.75) (xy 159.75 124.25)
+        (xy 154.5 129.5) (xy 144.25 129.5) (xy 143.5 129.5) (xy 143.5 129) (xy 144.25 129)
+        (xy 146.75 126.5) (xy 154.5 126.5) (xy 155.75 125.25) (xy 155.75 122) (xy 153 122)
+        (xy 153 112.75) (xy 143 112.75) (xy 143 118) (xy 126 118) (xy 126 112.75)
+        (xy 114.25 112.75) (xy 114.25 119.5) (xy 113.5 120.25) (xy 109 120.25) (xy 109 123.25)
+        (xy 103.5 123.25) (xy 103.5 120.25) (xy 102.25 120.25)
       )
     )

Commit message: updated pcb
Routing:
- net /SDA: track 5.40 -> 102.0 mm, vias 0 -> 2
- net /SCL: track 5.43 -> 92.0 mm, vias 0 -> 1
- net /PWM_B: track 0.00 -> 86.4 mm, vias 0 -> 2
- net /~AL: track 5.60 -> 86.9 mm, vias 0 -> 1
- net /~INT: track 5.51 -> 55.0 mm, vias 0 -> 1
- net /PWM_G: track 0.00 -> 42.5 mm, vias 0 -> 1
- net /PWM_R: track 0.00 -> 32.0 mm
- net /IR_Rx: track 0.00 -> 19.8 mm
- net GND: vias 20 -> 24

Commit message: updated pcb
Routing:
- net /charger/ADAPTER: track 191.2 -> 146.6 mm
- net Net-(D5-Pad1): track 25.3 -> 0.00 mm
- added copper zone on F.Cu, net /charger/ADAPTER
- added copper zone on F.Cu, net Net-(D5-Pad1)
Changed lines of the file:
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@@
     (thickness 1.6)
     (drawings 6)
-    (tracks 478)
+    (tracks 443)
     (zones 0)
     (modules 77)
@@
     (mod_text_size 1 1)
     (mod_text_width 0.15)
-    (pad_size 0.85 0.3)
-    (pad_drill 0)
+    (pad_size 4 4)
+    (pad_drill 2.2)
     (pad_to_mask_clearance 0.2)
     (aux_axis_origin 0 0)
@@
       (net 5 GND))
     (pad 1 thru_hole rect (at 0 -10.25 180) (size 4 4) (drill 2.2) (layers *.Cu *.Mask)
-      (net 8 "Net-(D5-Pad1)"))
+      (net 8 "Net-(D5-Pad1)") (zone_connect 2))
     (pad 2 thru_hole circle (at 0 -3.6 180) (size 4 4) (drill 2.2) (layers *.Cu *.Mask)
       (net 5 GND))
@@
       (net 8 "Net-(D5-Pad1)"))
     (pad 3 smd rect (at 0 1.2) (size 3.2 4.9) (layers F.Cu F.Mask)
-      (net 24 /charger/ADAPTER))
+      (net 24 /charger/ADAPTER) (zone_connect 2))
     (pad 1 smd rect (at -0.97 -3.15) (size 0.95 1) (layers F.Cu F.Paste F.Mask)
       (net 8 "Net-(D5-Pad1)"))
@@
   (segment (start 171.2 112.5) (end 172.5 112.5) (width 2) (layer B.Cu) (net 24))
   (segment (start 170 112.5) (end 171.2 112.5) (width 2) (layer B.Cu) (net 24))
-  (segment (start 171.2 112.5) (end 172.5 112.5) (width 2) (layer F.Cu) (net 24))
-  (segment (start 171.25 111.25) (end 171.25 110) (width 2) (layer F.Cu) (net 24))
-  (segment (start 172.5 111.25) (end 171.25 111.25) (width 2) (layer F.Cu) (net 24))
-  (segment (start 171.25 110) (end 172.5 110) (width 2) (layer F.Cu) (net 24))
-  (segment (start 170 110) (end 171.25 110) (width 2) (layer F.Cu) (net 24))
   (via (at 172.5 110) (size 0.8) (drill 0.4) (layers F.Cu B.Cu) (net 24))
   (via (at 171.25 110) (size 0.8) (drill 0.4) (layers F.Cu B.Cu) (net 24))
@@
   (via (at 172.5 111.25) (size 0.8) (drill 0.4) (layers F.Cu B.Cu) (net 24))
   (via (at 171.25 111.25) (size 0.8) (drill 0.4) (layers F.Cu B.Cu) (net 24))
-  (segment (start 170 111.25) (end 170 111.3) (width 2) (layer F.Cu) (net 24))
-  (segment (start 170 111.3) (end 171.2 112.5) (width 2) (layer F.Cu) (net 24))
   (via (at 171.2 112.5) (size 0.8) (drill 0.4) (layers F.Cu B.Cu) (net 24))
   (via (at 170 111.25) (size 0.8) (drill 0.4) (layers F.Cu B.Cu) (net 24))
-  (segment (start 171.65 108.45) (end 175.25 108.45) (width 2) (layer F.Cu) (net 24))
-  (segment (start 175.25 110.75) (end 173.5 112.5) (width 2) (layer F.Cu) (net 24))
-  (segment (start 173.5 112.5) (end 171.2 112.5) (width 2) (layer F.Cu) (net 24))
-  (segment (start 175.25 108.45) (end 175.25 110.75) (width 2) (layer F.Cu) (net 24))
-  (segment (start 172.75 108.45) (end 175.25 108.45) (width 2) (layer F.Cu) (net 24))
-  (segment (start 170 112.5) (end 170 111.25) (width 2) (layer F.Cu) (net 24))
-  (segment (start 170 111.2) (end 172.75 108.45) (width 2) (layer F.Cu) (net 24))
-  (segment (start 171.65 108.45) (end 172.75 108.45) (width 2) (layer F.Cu) (net 24))
-  (segment (start 170 111.25) (end 170 110.1) (width 2) (layer F.Cu) (net 24))
-  (segment (start 170 111.25) (end 170 111.2) (width 2) (layer F.Cu) (net 24))
-  (segment (start 170 110.1) (end 171.65 108.45) (width 2) (layer F.Cu) (net 24))
-  (segment (start 170 112.5) (end 171.2 112.5) (width 2) (layer F.Cu) (net 24))
-  (segment (start 171.2 112.5) (end 175.25 108.45) (width 2) (layer F.Cu) (net 24))
-  (segment (start 175.25 109.25) (end 172 112.5) (width 2) (layer F.Cu) (net 24))
-  (segment (start 172 112.5) (end 170 112.5) (width 2) (layer F.Cu) (net 24))
   (via (at 170 112.5) (size 0.8) (drill 0.4) (layers F.Cu B.Cu) (net 24))
   (segment (start 175.25 108.45) (end 175.25 109.25) (width 2) (layer F.Cu) (net 24))
@@
   (segment (start 155.25 94.3) (end 155.2 94.35) (width 1) (layer F.Cu) (net 4))
   (segment (start 161.943309 94.35) (end 161.95 94.343309) (width 1) (layer F.Cu) (net 4))
-  (segment (start 182 99) (end 178.82 99) (width 2) (layer F.Cu) (net 8))
-  (segment (start 178.82 99) (end 178 99.82) (width 2) (layer F.Cu) (net 8))
-  (segment (start 174.28 104.1) (end 174.28 102.72) (width 2) (layer F.Cu) (net 8))
-  (segment (start 174.28 102.72) (end 175.4 101.6) (width 2) (layer F.Cu) (net 8))
-  (segment (start 176.22 104.1) (end 176.22 101.6) (width 2) (layer F.Cu) (net 8))
-  (segment (start 176.22 101.6) (end 178 99.82) (width 2) (layer F.Cu) (net 8))
-  (segment (start 178 99.82) (end 178 99) (width 2) (layer F.Cu) (net 8))
-  (segment (start 174.28 104.1) (end 175.2 104.1) (width 2) (layer F.Cu) (net 8))
-  (segment (start 175.2 104.1) (end 176.22 104.1) (width 2) (layer F.Cu) (net 8))
-  (segment (start 175.4 101.6) (end 175.4 103.9) (width 2) (layer F.Cu) (net 8))
-  (segment (start 175.4 103.9) (end 175.2 104.1) (width 2) (layer F.Cu) (net 8))
-  (segment (start 182 99) (end 178 99) (width 2) (layer F.Cu) (net 8))
-  (segment (start 178 99) (end 175.4 101.6) (width 2) (layer F.Cu) (net 8))
   (segment (start 187.6 103.3) (end 184.68 103.3) (width 0.5) (layer F.Cu) (net 9))
   (segment (start 184.68 103.3) (end 184.38 103) (width 0.5) (layer F.Cu) (net 9))
@@
       )
     )
+  )
+  (zone (net 24) (net_name /charger/ADAPTER) (layer F.Cu) (hatch edge 0.508)
+    (priority 1)
+    (connect_pads (clearance 0.508))
+    (min_thickness 0.254)
+    (fill yes (arc_segments 16) (thermal_gap 0.508) (thermal_bridge_width 0.508))
+    (polygon
+      (pts
+        (xy 169.25 109.25) (xy 173 109.25) (xy 173 105.75) (xy 177.5 105.75) (xy 177.5 113.25)
+        (xy 169.25 113.25)
+      )
+    )
+  )
+  (zone (net 8) (net_name "Net-(D5-Pad1)") (layer F.Cu) (hatch edge 0.508)
+    (priority 2)
+    (connect_pads (clearance 0.508))
+    (min_thickness 0.254)
+    (fill yes (arc_segments 16) (thermal_gap 0.508) (thermal_bridge_width 0.508))
+    (polygon
+      (pts
+        (xy 173 102.75) (xy 179.25 96.5) (xy 184.5 96.5) (xy 184.5 101.5) (xy 179.25 101.5)
+        (xy 177.5 103.25) (xy 177.5 105.25) (xy 173 105.25)
+      )
+    )

Commit message: updated pcb
Routing:
- net /charger/ADAPTER: track 146.6 -> 15.4 mm
- net /PWM_R: track 32.0 -> 52.9 mm, vias 0 -> 2
- net /PWM_G: track 42.5 -> 58.8 mm, vias 1 -> 3
- net /PWM_B: track 86.4 -> 70.4 mm, vias 2 -> 3
- added copper zone on B.Cu, net /charger/ADAPTER

Commit message: updated pcb
Routing:
- net /~AL: track 86.9 -> 5.60 mm, vias 1 -> 0
- net /~INT: track 55.0 -> 5.51 mm, vias 1 -> 0
- net /SDA: track 102.0 -> 53.8 mm
- net /SCL: track 92.0 -> 45.8 mm, vias 1 -> 0
- net /PWM_R: track 52.9 -> 72.8 mm, vias 2 -> 3
- net /PWM_G: track 58.8 -> 71.8 mm
- net /PWM_B: track 70.4 -> 74.7 mm
- net Net-(C19-Pad1): track 17.9 -> 22.0 mm
