File: hw/back.kicad_pcb (KiCad board)
At the start: 2 copper layers, 110 x 55 mm, 77 parts, among them J1 IDC_02X13, J2 FC681495, J3 N42GK-04, Q1 BSC080N03MS, U1 OSRB38C9BA, U2 MCP1826S, U3 MCP1826S, U4 BQ24192, U5 LTC1871, U6 LTC2941CMS8E

Commit message: updated pcb
Routing:
- net /IR_Rx: track 20.7 -> 28.5 mm
- net +3V3: track 62.8 -> 66.8 mm
Changed lines of the file:
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@@
     (thickness 1.6)
     (drawings 6)
-    (tracks 518)
+    (tracks 520)
     (zones 0)
     (modules 77)
@@
   (segment (start 139.163589 129.95) (end 139.275 129.95) (width 0.25) (layer F.Cu) (net 10))
   (segment (start 136 133) (end 137 133) (width 0.25) (layer F.Cu) (net 10))
-  (segment (start 136.649999 93.100001) (end 136.25 93.5) (width 1) (layer B.Cu) (net 11))
-  (segment (start 136.25 94.065685) (end 136.25 93.5) (width 1) (layer F.Cu) (net 11))
-  (segment (start 132.5 98.13) (end 134.2 98.13) (width 1) (layer F.Cu) (net 11))
-  (via (at 136.25 93.5) (size 0.8) (drill 0.4) (layers F.Cu B.Cu) (net 11))
-  (segment (start 134.2 98.13) (end 136.25 96.08) (width 1) (layer F.Cu) (net 11))
-  (segment (start 167.250018 89.75) (end 140 89.75) (width 1) (layer B.Cu) (net 11))
-  (segment (start 171 93.499982) (end 167.250018 89.75) (width 1) (layer B.Cu) (net 11))
-  (segment (start 140 89.75) (end 136.649999 93.100001) (width 1) (layer B.Cu) (net 11))
-  (segment (start 136.25 96.08) (end 136.25 94.065685) (width 1) (layer F.Cu) (net 11))
+  (segment (start 132.5 98.13) (end 135.37 98.13) (width 1) (layer F.Cu) (net 11))
+  (segment (start 137.25 96.25) (end 137.25 89.065689) (width 1) (layer F.Cu) (net 11))
+  (segment (start 137.25 89.065689) (end 137.25 88.500004) (width 1) (layer F.Cu) (net 11))
+  (segment (start 135.37 98.13) (end 137.25 96.25) (width 1) (layer F.Cu) (net 11))
+  (via (at 137.25 88.500004) (size 0.8) (drill 0.4) (layers F.Cu B.Cu) (net 11))
+  (segment (start 166.000022 88.500004) (end 137.815685 88.500004) (width 1) (layer B.Cu) (net 11))
+  (segment (start 171 93.499982) (end 166.000022 88.500004) (width 1) (layer B.Cu) (net 11))
+  (segment (start 137.815685 88.500004) (end 137.25 88.500004) (width 1) (layer B.Cu) (net 11))
   (segment (start 171 92.373309) (end 171 92.934297) (width 1) (layer F.Cu) (net 11))
   (segment (start 171 92.934297) (end 171 93.499982) (width 1) (layer F.Cu) (net 11))
@@
   (segment (start 135.88 126) (end 136.825 126) (width 0.25) (layer F.Cu) (net 24))
   (via (at 138 126.5) (size 0.8) (drill 0.4) (layers F.Cu B.Cu) (net 24))
-  (via (at 143.75 94) (size 0.8) (drill 0.4) (layers F.Cu B.Cu) (net 3))
-  (via (at 142.5 94) (size 0.8) (drill 0.4) (layers F.Cu B.Cu) (net 3))
-  (via (at 142.5 95.25) (size 0.8) (drill 0.4) (layers F.Cu B.Cu) (net 3))
-  (via (at 143.75 95.25) (size 0.8) (drill 0.4) (layers F.Cu B.Cu) (net 3))
+  (via (at 143.75 96) (size 0.8) (drill 0.4) (layers F.Cu B.Cu) (net 3))
+  (via (at 142.5 96) (size 0.8) (drill 0.4) (layers F.Cu B.Cu) (net 3))
+  (via (at 142.5 97) (size 0.8) (drill 0.4) (layers F.Cu B.Cu) (net 3))
+  (via (at 143.75 97) (size 0.8) (drill 0.4) (layers F.Cu B.Cu) (net 3))
   (via (at 142.97501 128.55) (size 0.8) (drill 0.4) (layers F.Cu B.Cu) (net 5))
   (via (at 142.97501 129.85) (size 0.8) (drill 0.4) (layers F.Cu B.Cu) (net 5))
@@
   (segment (start 138.74 123.43) (end 138 123.43) (width 0.25) (layer F.Cu) (net 34))
   (segment (start 140.794682 125.988985) (end 140.794682 125.484682) (width 0.25) (layer F.Cu) (net 34))
-  (segment (start 137.75 96.75) (end 137.75 92.75) (width 0.5) (layer F.Cu) (net 35))
-  (segment (start 142.46 101.46) (end 137.75 96.75) (width 0.5) (layer F.Cu) (net 35))
-  (segment (start 142.46 107.5) (end 142.46 101.46) (width 0.5) (layer F.Cu) (net 35))
-  (segment (start 137.75 92.75) (end 136 91) (width 0.5) (layer F.Cu) (net 35))
-  (segment (start 136 91) (end 134.48 91) (width 0.5) (layer F.Cu) (net 35))
+  (segment (start 138 87.5) (end 136.656484 87.5) (width 0.5) (layer F.Cu) (net 35))
+  (segment (start 138.75 105.29) (end 138.75 88.25) (width 0.5) (layer F.Cu) (net 35))
+  (segment (start 138.75 88.25) (end 138 87.5) (width 0.5) (layer F.Cu) (net 35))
+  (segment (start 136.049991 89.430009) (end 134.48 91) (width 0.5) (layer F.Cu) (net 35))
+  (segment (start 140.96 107.5) (end 138.75 105.29) (width 0.5) (layer F.Cu) (net 35))
+  (segment (start 136.656484 87.5) (end 136.049991 88.106493) (width 0.5) (layer F.Cu) (net 35))
+  (segment (start 136.049991 88.106493) (end 136.049991 89.430009) (width 0.5) (layer F.Cu) (net 35))
+  (segment (start 142.46 107.5) (end 140.96 107.5) (width 0.5) (layer F.Cu) (net 35))
   (segment (start 104.05 125.75) (end 102.573004 125.75) (width 0.25) (layer F.Cu) (net 36))
   (segment (start 102.573004 125.75) (end 100.63 125.75) (width 0.25) (layer F.Cu) (net 36))
@@
     (polygon
       (pts
-        (xy 147.25 96.25) (xy 147.25 93.25) (xy 144.75 93.25) (xy 144.75 91.25) (xy 140.5 91.25)
-        (xy 140.5 96.25)
+        (xy 147.25 97.5) (xy 147.25 93.25) (xy 144.75 93.25) (xy 144.75 91.25) (xy 140.5 91.25)
+        (xy 140.5 97.5)
       )
     )
@@
       (pts
         (xy 125.5 135.75) (xy 129 135.75) (xy 129 130.5) (xy 109.5 111) (xy 109.5 101)
-        (xy 113 97.5) (xy 145 97.5) (xy 145 92.75) (xy 141.25 92.75) (xy 141.25 95.5)
-        (xy 113 95.5) (xy 113 88.25) (xy 104 88.25) (xy 104 89.5) (xy 105.5 89.5)
-        (xy 105.5 110.5) (xy 125.5 130.5)
+        (xy 113 97.5) (xy 144.25 97.5) (xy 144.25 95.5) (xy 141.25 95.5) (xy 113 95.5)
+        (xy 113 88.25) (xy 104 88.25) (xy 104 89.5) (xy 105.5 89.5) (xy 105.5 110.5)
+        (xy 125.5 130.5)
       )
     )

Commit message: updated pcb
Routing:
- net /PWM_R: vias 4 -> 6
- net /PWM_G: vias 4 -> 6
- net /PWM_B: vias 4 -> 6
Changed lines of the file:
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@@
     (thickness 1.6)
     (drawings 6)
-    (tracks 520)
+    (tracks 534)
     (zones 0)
     (modules 77)
@@
   (segment (start 170.156691 94.343309) (end 171 93.5) (width 1) (layer F.Cu) (net 11))
   (segment (start 171 93.5) (end 171 92.073309) (width 1) (layer F.Cu) (net 11))
+  (segment (start 140.75 101.75) (end 169.25 101.75) (width 0.5) (layer B.Cu) (net 12))
+  (segment (start 134 101.75) (end 140.75 101.75) (width 0.5) (layer F.Cu) (net 12))
+  (via (at 140.75 101.75) (size 0.8) (drill 0.4) (layers F.Cu B.Cu) (net 12))
+  (segment (start 124.5 101.75) (end 134 101.75) (width 0.5) (layer B.Cu) (net 12))
+  (via (at 134 101.75) (size 0.8) (drill 0.4) (layers F.Cu B.Cu) (net 12))
   (segment (start 121.78 91) (end 121.78 93.47) (width 0.5) (layer F.Cu) (net 12))
   (segment (start 121.78 93.47) (end 119.25 96) (width 0.5) (layer F.Cu) (net 12))
@@
   (segment (start 171.5 107.75) (end 171.5 106) (width 0.5) (layer F.Cu) (net 12))
   (segment (start 169.25 101.75) (end 171.5 104) (width 0.5) (layer B.Cu) (net 12))
-  (segment (start 124.5 101.75) (end 169.25 101.75) (width 0.5) (layer B.Cu) (net 12))
   (segment (start 171.5 104) (end 171.5 105.434315) (width 0.5) (layer B.Cu) (net 12))
   (segment (start 121.25 105) (end 124.5 101.75) (width 0.5) (layer B.Cu) (net 12))
   (segment (start 171.5 105.434315) (end 171.5 106) (width 0.5) (layer B.Cu) (net 12))
+  (segment (start 140.75 103) (end 168.25 103) (width 0.5) (layer B.Cu) (net 15))
+  (segment (start 134 103) (end 140.75 103) (width 0.5) (layer F.Cu) (net 15))
+  (via (at 140.75 103) (size 0.8) (drill 0.4) (layers F.Cu B.Cu) (net 15))
+  (segment (start 125.25 103) (end 134 103) (width 0.5) (layer B.Cu) (net 15))
+  (via (at 134 103) (size 0.8) (drill 0.4) (layers F.Cu B.Cu) (net 15))
   (segment (start 118 95.5) (end 118 102.25) (width 0.5) (layer F.Cu) (net 15))
   (segment (start 119.24 94.26) (end 118 95.5) (width 0.5) (layer F.Cu) (net 15))
@@
   (segment (start 115.649999 104.600001) (end 115.25 105) (width 0.5) (layer F.Cu) (net 15))
   (segment (start 121.25 107) (end 125.25 103) (width 0.5) (layer B.Cu) (net 15))
-  (segment (start 125.25 103) (end 168.25 103) (width 0.5) (layer B.Cu) (net 15))
   (segment (start 168.25 103) (end 170.25 105) (width 0.5) (layer B.Cu) (net 15))
   (segment (start 170.25 105) (end 170.25 107.000006) (width 0.5) (layer B.Cu) (net 15))
+  (segment (start 140.75 104.25) (end 167.241995 104.25) (width 0.5) (layer B.Cu) (net 16))
+  (segment (start 167.241995 104.25) (end 167.991995 105) (width 0.5) (layer B.Cu) (net 16))
+  (segment (start 134 104.25) (end 140.75 104.25) (width 0.5) (layer F.Cu) (net 16))
+  (via (at 140.75 104.25) (size 0.8) (drill 0.4) (layers F.Cu B.Cu) (net 16))
+  (segment (start 126 104.25) (end 134 104.25) (width 0.5) (layer B.Cu) (net 16))
+  (via (at 134 104.25) (size 0.8) (drill 0.4) (layers F.Cu B.Cu) (net 16))
   (segment (start 115.25 103) (end 116.7 101.55) (width 0.5) (layer F.Cu) (net 16))
   (segment (start 116.7 94.8) (end 116.7 91) (width 0.5) (layer F.Cu) (net 16))
   (segment (start 116.7 101.55) (end 116.7 94.8) (width 0.5) (layer F.Cu) (net 16))
   (segment (start 121.25 109) (end 126 104.25) (width 0.5) (layer B.Cu) (net 16))
-  (segment (start 126 104.25) (end 167.241995 104.25) (width 0.5) (layer B.Cu) (net 16))
-  (segment (start 167.241995 104.25) (end 167.991995 105) (width 0.5) (layer B.Cu) (net 16))
   (segment (start 163.75 127.5) (end 164.25 128) (width 0.25) (layer F.Cu) (net 20))
   (segment (start 163.275 127.5) (end 163.75 127.5) (width 0.25) (layer F.Cu) (net 20))
@@
   (segment (start 138.74 123.43) (end 138 123.43) (width 0.25) (layer F.Cu) (net 34))
   (segment (start 140.794682 125.988985) (end 140.794682 125.484682) (width 0.25) (layer F.Cu) (net 34))
+  (segment (start 138.75 99) (end 138.75 88.25) (width 0.5) (layer F.Cu) (net 35))
+  (segment (start 140.75 100) (end 139.75 100) (width 0.5) (layer F.Cu) (net 35))
+  (segment (start 139.75 100) (end 138.75 99) (width 0.5) (layer F.Cu) (net 35))
+  (segment (start 142.46 101.71) (end 140.75 100) (width 0.5) (layer F.Cu) (net 35))
+  (segment (start 142.46 107.5) (end 142.46 101.71) (width 0.5) (layer F.Cu) (net 35))
   (segment (start 138 87.5) (end 136.656484 87.5) (width 0.5) (layer F.Cu) (net 35))
-  (segment (start 138.75 105.29) (end 138.75 88.25) (width 0.5) (layer F.Cu) (net 35))
   (segment (start 138.75 88.25) (end 138 87.5) (width 0.5) (layer F.Cu) (net 35))
   (segment (start 136.049991 89.430009) (end 134.48 91) (width 0.5) (layer F.Cu) (net 35))
-  (segment (start 140.96 107.5) (end 138.75 105.29) (width 0.5) (layer F.Cu) (net 35))
   (segment (start 136.656484 87.5) (end 136.049991 88.106493) (width 0.5) (layer F.Cu) (net 35))
   (segment (start 136.049991 88.106493) (end 136.049991 89.430009) (width 0.5) (layer F.Cu) (net 35))
-  (segment (start 142.46 107.5) (end 140.96 107.5) (width 0.5) (layer F.Cu) (net 35))
   (segment (start 104.05 125.75) (end 102.573004 125.75) (width 0.25) (layer F.Cu) (net 36))
   (segment (start 102.573004 125.75) (end 100.63 125.75) (width 0.25) (layer F.Cu) (net 36))

Commit message: updated pcb
Routing:
- net /~AL: track 5.60 -> 122.3 mm, vias 0 -> 1
- net /SDA: track 53.1 -> 133.1 mm
- net /SCL: track 45.2 -> 123.9 mm, vias 0 -> 1
- net /~INT: track 5.51 -> 83.1 mm, vias 0 -> 1

Commit message: updated pcb
Routing:
- net /SCL: track 123.9 -> 121.1 mm
- net /SDA: track 133.1 -> 130.8 mm
- net /~AL: track 122.3 -> 121.0 mm
- net /~INT: track 83.1 -> 82.2 mm
- net Net-(C19-Pad1): track 22.7 -> 23.3 mm

Commit message: updated pcb
Routing:
- net /PWM_B: track 108.9 -> 107.8 mm
- net /~AL: track 121.0 -> 121.8 mm
Other:
- net class Default: clearance 0.2 -> 0.1
- rule trace_clearance: 0.2 -> 0.1
